File: PCBs/arduino_mega_shield/arduino_mega_shield_integrated.kicad_sch (KiCad schematic)
At the start: 42 parts, among them J1 to_common_anode_RGB_LED1, J10 to_common_anode_RGB_LED1, J11 Barrel_Jack_Switch_Pin3Ring, J13 to_fan, J14 to_common_anode_RGB_LED1, J15 to_common_anode_RGB_LED1, J2 to_common_anode_RGB_LED1, J3 to_common_anode_RGB_LED1, J4 to_UNO, J5 to_radius_switch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

Commit message: finish schematics for mega board, and fix error in spreadsheet
Parts:
- removed C1: C_Small, symbol Device:C_Small
- removed J10, J7, J8: to_common_anode_RGB_LED1, symbol Connector:Conn_01x04_Socket
- removed J11: Barrel_Jack_Switch_Pin3Ring, symbol Connector:Barrel_Jack_Switch_Pin3Ring
- removed J4: to_UNO, symbol Connector:Conn_01x06_Socket
- removed J6: to_stepper_driver, symbol Connector:Conn_01x07_Socket
- removed R19, R24: 10k, symbol Device:R_Small
- removed R20, R21, R25: 220, symbol Device:R_Small
- removed R22: 330, symbol Device:R_Small
- removed R23: 1k, symbol Device:R_Small
- removed U1: LM350_TO220, Package_TO_SOT_THT:TO-220-3_Vertical, symbol Regulator_Linear:LM350_TO220
- added J10: to_start_pushbutton, symbol Connector:Conn_01x02_Socket
- added J11: to_cycle_pushbutton, symbol Connector:Conn_01x02_Socket
- added J12: to_kill_pushbutton, symbol Connector:Conn_01x02_Socket
- added J4, J6, J7, J8: to_IR_sensor, symbol Connector:Conn_01x03_Socket
- J5: value to_radius_switch -> to_IR_sensor
- R3: value 220 -> 10k
Connections:
- net +5V: now also A1.5V1 (5V), A1.5V3 (5V), A1.5V4 (5V); no longer J13.1 (Pin_1), J5.1 (Pin_1), J9.7 (Pin_7), R3.1
- net GND: now also R3.2, J10.2 (Pin_2), J11.2 (Pin_2), J12.2 (Pin_2); no longer J13.2 (Pin_2), J5.3 (Pin_3), J9.8 (Pin_8)
- net at A1.D2 (D2_INT0), R4.1: now also J12.1 (Pin_1)
- net at A1.D22: now also R3.1, J11.1 (Pin_1); no longer R2.1
- net at A1.D24: now also R2.1, J10.1 (Pin_1)
- net +12V: no longer names the net of A1.VIN
- net pin23: no longer names the net of A1.D23
- net to_uno1: no longer names the net of A1.D3 (D3_INT1)
- net to_uno2: no longer names the net of A1.D18 (D18/TX1)
- net to_uno3: no longer names the net of A1.D19 (D19/RX1)
- net to_uno4: no longer names the net of A1.D20 (D20/SDA)
- net to_uno5: no longer names the net of A1.D21 (D21/SCL)
- no-connect marks 53 -> 0
Other:
- moved on the sheet: J13
